Commit message: Added a contact sensor to the chassis of the erle rover and fixed the collision box for their chassis graphic

File: ardupilot_sitl_gazebo_plugin/ardupilot_sitl_gazebo_plugin/urdf/base_rover.urdf (robot description, URDF)
Before this commit: robot rover, 7 links, 6 joints
Links:
- link chassis: geometry collision box size=0.55 0.2 0.012; visual mesh filename=package://ardupilot_sitl_gazebo_plugin/meshes/meshes_rover/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 scale=0.0011 0.0011 0.0011

File: ardupilot_sitl_gazebo_plugin/ardupilot_sitl_gazebo_plugin/urdf/rover.urdf (robot description, URDF)
Before this commit: robot rover, 7 links, 6 joints
Links:
- link chassis: geometry collision box size=0.55 0.2 0.012; visual mesh filename=package://ardupilot_sitl_gazebo_plugin/meshes/meshes_rover/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 scale=0.0011 0.0011 0.0011

Commit message: Finished integrating the contact sensor in the chassis into the evo-ros framework

File: ardupilot_sitl_gazebo_plugin/ardupilot_sitl_gazebo_plugin/urdf/base_rover.urdf (robot description, URDF)
Before this commit: robot rover, 7 links, 6 joints
Links:
- link chassis: geometry collision box size=0.65 0.2 0.02; visual mesh filename=package://ardupilot_sitl_gazebo_plugin/meshes/meshes_rover/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 scale=0.0011 0.0011 0.0011

File: ardupilot_sitl_gazebo_plugin/ardupilot_sitl_gazebo_plugin/urdf/rover.urdf (robot description, URDF)
Before this commit: robot rover, 7 links, 6 joints
Links:
- link chassis: geometry collision box size=0.65 0.2 0.02; visual mesh filename=package://ardupilot_sitl_gazebo_plugin/meshes/meshes_rover/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 scale=0.0011 0.0011 0.0011

File: ardupilot_sitl_gazebo_plugin/ardupilot_sitl_gazebo_plugin/urdf/simongle-XPS-13-V14_rover.urdf (robot description, URDF)
Before this commit: robot rover, 7 links, 6 joints
Links:
- link chassis: geometry collision box size=0.65 0.2 0.02; visual mesh filename=package://ardupilot_sitl_gazebo_plugin/meshes/meshes_rover/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 scale=0.0011 0.0011 0.0011
