Commit message: Updating because i haven't in forever

File: ardupilot_sitl_gazebo_plugin/ardupilot_sitl_gazebo_plugin/urdf/gps_home_location.xacro (robot description, xacro)
@@ -1,9 +1,9 @@
 <?xml version="1.0"?>
 <!-- File auto-generated by sim_vehicle.sh -->
-<!-- Location at CMAC -->
+<!-- Location at MSU-EB -->
 <robot xmlns:xacro="http://ros.org/wiki/xacro">
   <!-- The following GPS coordinates locate the center of Gazebo's map -->
-  <xacro:property name="referenceLatitude" value="-35.363261" />     <!-- in degrees -->
-  <xacro:property name="referenceLongitude" value="149.165230" />   <!-- in degrees -->
-  <xacro:property name="referenceAltitude" value="584" />     <!-- in meters above sea level -->
+  <xacro:property name="referenceLatitude" value="42.724908" />     <!-- in degrees -->
+  <xacro:property name="referenceLongitude" value="-84.480979" />   <!-- in degrees -->
+  <xacro:property name="referenceAltitude" value="0" />     <!-- in meters above sea level -->
 </robot>

File: ardupilot_sitl_gazebo_plugin/ardupilot_sitl_gazebo_plugin/urdf/sensors/hector_sonar_sensor.urdf.xacro (robot description, xacro)
@@ -1,5 +1,5 @@
 <?xml version="1.0"?>
 <robot xmlns:xacro="http://ros.org/wiki/xacro">
-  <xacro:macro name="sonar_sensor" params="name parent *origin ros_topic update_rate min_range max_range field_of_view ray_count sensor_mesh">
+  <xacro:macro name="sonar_sensor" params="name parent *origin ros_topic update_rate min_range max_range field_of_view ray_count">
     <joint name="${name}_joint" type="fixed">
       <xacro:insert_block name="origin" />
@@ -17,16 +17,13 @@
         <geometry>
           <!--<box size="0.01 0.01 0.01" /> -->
-          <!-- <mesh filename="package://rotors_description/meshes/sonar_sensor/max_sonar_ez4.dae"/> -->
-           <!--<mesh filename="package://ardupilot_sitl_gazebo_plugin/meshes/${sensor_mesh}"/>-->
-           <mesh filename="model://${sensor_mesh}"/>
-         <!-- <mesh filename="package://ardupilot_sitl_gazebo_plugin/meshes/lidar_lite_v2/meshes/lidar_lite_v2.dae"/> -->
+          <mesh filename="package://hector_sensors_description/meshes/sonar_sensor/max_sonar_ez4.dae"/>
         </geometry>
       </visual>
-   <!--   <collision>
+      <collision>
         <origin xyz="0 0 0" rpy="0 0 0" />
         <geometry>
           <box size="0.01 0.01 0.01" />
         </geometry>
-      </collision> -->
+      </collision>
     </link>
     <gazebo reference="${name}_link">
@@ -35,5 +32,5 @@
         <update_rate>${update_rate}</update_rate>
         <pose>0 0 0 0 0 0</pose>
-        <visualize>true</visualize>
+        <visualize>false</visualize>
         <ray>
           <scan>
@@ -47,6 +44,6 @@
               <samples>${ray_count}</samples>
               <resolution>1</resolution>
-              <min_angle>-${field_of_view/2}</min_angle>
-              <max_angle>${field_of_view/2}</max_angle>
+              <min_angle>-1</min_angle>
+              <max_angle>1</max_angle>
             </vertical>
           </scan>
@@ -57,6 +54,5 @@
           </range>
         </ray>
-       <!-- plugin name="gazebo_ros_${name}_controller" filename="librotors_gazebo_sonar_plugin.so"> -->
-		<plugin name="gazebo_ros_${name}_controller" filename="libhector_gazebo_ros_sonar.so">
+        <plugin name="gazebo_ros_${name}_controller" filename="libhector_gazebo_ros_sonar.so">
           <gaussianNoise>0.005</gaussianNoise>
           <topicName>${ros_topic}</topicName>

File: ardupilot_sitl_gazebo_plugin/ardupilot_sitl_gazebo_plugin/urdf/sensors/lidar_sensor.urdf.xacro (robot description, xacro)
@@ -56,5 +56,6 @@
           </range>
         </ray>
-        <plugin name="gazebo_ros_${name}_controller" filename="librotors_gazebo_sonar_plugin.so">
+       <!-- plugin name="gazebo_ros_${name}_controller" filename="librotors_gazebo_sonar_plugin.so"> -->
+		<plugin name="gazebo_ros_${name}_controller" filename="libhector_gazebo_ros_sonar.so">
           <gaussianNoise>0.005</gaussianNoise>
           <topicName>${ros_topic}</topicName>

Commit message: Continuing progress to get the sonar placement run ready. Working on comminication between controller and sim manager and clean resets

File: ardupilot_sitl_gazebo_plugin/ardupilot_sitl_gazebo_plugin/urdf/gps_home_location.xacro (robot description, xacro)
@@ -1,9 +1,9 @@
 <?xml version="1.0"?>
 <!-- File auto-generated by sim_vehicle.sh -->
-<!-- Location at MSU-EB -->
+<!-- Location at CMAC -->
 <robot xmlns:xacro="http://ros.org/wiki/xacro">
   <!-- The following GPS coordinates locate the center of Gazebo's map -->
-  <xacro:property name="referenceLatitude" value="42.724908" />     <!-- in degrees -->
-  <xacro:property name="referenceLongitude" value="-84.480979" />   <!-- in degrees -->
-  <xacro:property name="referenceAltitude" value="0" />     <!-- in meters above sea level -->
+  <xacro:property name="referenceLatitude" value="-35.363261" />     <!-- in degrees -->
+  <xacro:property name="referenceLongitude" value="149.165230" />   <!-- in degrees -->
+  <xacro:property name="referenceAltitude" value="584" />     <!-- in meters above sea level -->
 </robot>
