Commit message: Added sensor knockout functionality

File: ardupilot_sitl_gazebo_plugin/ardupilot_sitl_gazebo_plugin/urdf/early_double_optimal_run1.urdf (robot description, URDF)
Before this commit: robot rover, 7 links, 6 joints
Joints:
- joint front_left_steering_joint: limit lower=-0.7727 upper=0.7727 effort=10.0 velocity=0.0 -> lower=-0.7727 upper=0.7727 effort=20.0 velocity=0.0
- joint front_left_wheel_joint: limit lower=0 upper=0 effort=10.0 velocity=0 -> lower=0 upper=0 effort=20.0 velocity=0
- joint front_right_steering_joint: limit lower=-0.7727 upper=0.7727 effort=10.0 velocity=0.0 -> lower=-0.7727 upper=0.7727 effort=20.0 velocity=0.0

File: ardupilot_sitl_gazebo_plugin/ardupilot_sitl_gazebo_plugin/urdf/single_optimal_run1.urdf (robot description, URDF)
Before this commit: robot rover, 7 links, 6 joints
Joints:
- joint front_left_steering_joint: limit lower=-0.7727 upper=0.7727 effort=10.0 velocity=0.0 -> lower=-0.7727 upper=0.7727 effort=20.0 velocity=0.0
- joint front_left_wheel_joint: limit lower=0 upper=0 effort=10.0 velocity=0 -> lower=0 upper=0 effort=20.0 velocity=0
- joint front_right_steering_joint: limit lower=-0.7727 upper=0.7727 effort=10.0 velocity=0.0 -> lower=-0.7727 upper=0.7727 effort=20.0 velocity=0.0
